File: Electronics/IDP_circuit_diagram_v1.sch (EAGLE design)
At the start: 33 parts, among them Q1 ARDUINOR3-NOIOREF-NOTEXT

Commit message: updated circuit diagram
Parts:
- removed DIST_SENSOR: HC-SR04, IDP_library:HC-SR04
- added BLOCK_SORTER, TUNNEL_SENSOR: HC-SR04, IDP_library:HC-SR04
Connections:
- new net N$1: BLOCK_SORTER.ECHO, Q1.D6
- new net N$3: BLOCK_SORTER.TRIG, Q1.D7
- net +5V: now also BLOCK_SORTER.VCC, TUNNEL_SENSOR.VCC; no longer DIST_SENSOR.VCC
- net GND: now also BLOCK_SORTER.GND, TUNNEL_SENSOR.GND; no longer DIST_SENSOR.GND
- net N$19: now also Q1.D10; no longer Q1.D9
- net N$20: now also Q1.D9, TUNNEL_SENSOR.TRIG; no longer DIST_SENSOR.TRIG, Q1.D8
- net N$36: now also Q1.D8, TUNNEL_SENSOR.ECHO; no longer DIST_SENSOR.ECHO, Q1.D7
- net N$57: now also Q1.A0
Other:
- moved on the sheet: GRABBER_SERVO, LED1, LED2, LED3, LED4, R12, R3, R6, R9

Commit message: updated schematic
Parts:
- added R16: 10 kΩ, IDP_library:R-EU_0204/2V
- added S1: MOMENTARY-SWITCH-SPST-PTH-6.0MM, SparkFun-Switches:MOMENTARY-SWITCH-SPST-PTH-6.0MM
Connections:
- removed net N$1: BLOCK_SORTER.ECHO, Q1.D6
- removed net N$19: GRABBER_SERVO.2, Q1.D10
- removed net N$36: Q1.D8, TUNNEL_SENSOR.ECHO
- removed net N$57: LEFT.3, Q1.A0, R2.1, SCHMITT1A.I
- new net N$2: LEFT.3, Q1.A3, R2.1, SCHMITT1A.I
- new net N$4: Q1.D2, R16.1, S1.2
- new net N$6: GRABBER_SERVO.2, Q1.D8
- new net N$8: Q1.D10, TUNNEL_SENSOR.ECHO
- new net N$9: BLOCK_SORTER.ECHO, Q1.D7
- net +5V: now also S1.1
- net GND: now also R16.2; no longer Q1.GND1
- net N$17: now also Q1.A0
- net N$3: now also Q1.D6; no longer Q1.D7
- net N$43: now also Q1.A1
- net N$44: no longer Q1.D5
- net N$49: now also Q1.A2
- net N$50: no longer Q1.D4
- net N$52: no longer Q1.D3
- net N$58: no longer Q1.D2
Other:
- moved on the sheet: LED1, LED2, LED3, LED4, R12, R3, R6, R9, SCHMITT1A, SCHMITT2A, SCHMITT3A, SCHMITT4A
